File: PLC_RaspberryPico2.kicad_pcb (KiCad board)
At the start: 2 copper layers, 25 parts, among them J1 Salidas Digitales a Reles, J10 ID1, J11 Alimentacion, J12 ID2, J2 ID1, J3 ID2, J4 ID3, J5 ID4, J6 ID5, J7 ID6, J8 ID7, J9 ID8, SW1 SW_Push, SW2 SW_Push, SW3 SW_Push, SW4 SW_Push

Commit message: 2 de Octubre
Parts:
- removed J10: ID1, TerminalBlock:TerminalBlock_MaiXu_MX126-5.0-03P_1x03_P5.00mm
- added A1: RaspberryPi_Pico, Module:RaspberryPi_Pico_Common_THT, F.Cu at (46.4, 116.3)
- added Alimentación1: Alimentacion, Connector_BarrelJack:BarrelJack_CUI_PJ-079BH_Horizontal, F.Cu at (131.8, 85.3)
- added G***: LOGO, Propia:Huella_PCB_SL_chica, F.Cu at (61.4, 74.0)
- added G***: LOGO, Propia:Huella_PCB_SL_chica, F.Cu at (62.2, 188.3)
- added I2C1: Display I2C, Connector_PinHeader_2.54mm:PinHeader_1x04_P2.54mm_Vertical, F.Cu at (48.6, 81.0)
- added I2C1: Display I2C, Connector_PinHeader_2.54mm:PinHeader_1x04_P2.54mm_Vertical, F.Cu at (49.4, 195.3)
- added IA1: IA2, TerminalBlock:TerminalBlock_MaiXu_MX126-5.0-03P_1x03_P5.00mm, F.Cu at (50.9, 44.6)
- added ID1: ID1, TerminalBlock:TerminalBlock_MaiXu_MX126-5.0-03P_1x03_P5.00mm, F.Cu at (137.5, 77.1)
- added ID2: ID2, TerminalBlock:TerminalBlock_MaiXu_MX126-5.0-03P_1x03_P5.00mm, F.Cu at (137.7, 59.6)
- added ID3: ID3, TerminalBlock:TerminalBlock_MaiXu_MX126-5.0-03P_1x03_P5.00mm, F.Cu at (137.7, 41.7)
- added ID4: ID4, TerminalBlock:TerminalBlock_MaiXu_MX126-5.0-03P_1x03_P5.00mm, F.Cu at (128.8, 33.0)
- added ID5: ID5, TerminalBlock:TerminalBlock_MaiXu_MX126-5.0-03P_1x03_P5.00mm, F.Cu at (111.2, 33.0)
- added ID6: ID6, TerminalBlock:TerminalBlock_MaiXu_MX126-5.0-03P_1x03_P5.00mm, F.Cu at (93.7, 33.0)
- added ID7: ID7, TerminalBlock:TerminalBlock_MaiXu_MX126-5.0-03P_1x03_P5.00mm, F.Cu at (76.7, 33.0)
- added ID8: ID8, TerminalBlock:TerminalBlock_MaiXu_MX126-5.0-03P_1x03_P5.00mm, F.Cu at (59.5, 33.0)
- added J13: OA1, TerminalBlock:TerminalBlock_MaiXu_MX126-5.0-02P_1x02_P5.00mm, F.Cu at (139.0, 221.7)
- added J13: OA1, TerminalBlock:TerminalBlock_MaiXu_MX126-5.0-02P_1x02_P5.00mm, F.Cu at (138.2, 107.3)
- added J14: OA2, TerminalBlock:TerminalBlock_MaiXu_MX126-5.0-02P_1x02_P5.00mm, F.Cu at (138.1, 121.1)
- added J14: OA2, TerminalBlock:TerminalBlock_MaiXu_MX126-5.0-02P_1x02_P5.00mm, F.Cu at (138.9, 235.4)
- added MCP6002: MCP6002-xMC, Package_DIP:DIP-8_W7.62mm_Socket_LongPads, F.Cu at (102.1, 223.1)
- added MCP6002: MCP6002-xMC, Package_DIP:DIP-8_W7.62mm_Socket_LongPads, F.Cu at (101.3, 108.8)
- added OD1: Salidas Digitales a Reles, Connector_PinHeader_2.54mm:PinHeader_1x10_P2.54mm_Vertical, F.Cu at (64.2, 122.6)
- added R1: 4k7, Resistor_THT:R_Axial_DIN0204_L3.6mm_D1.6mm_P7.62mm_Horizontal, F.Cu at (110.4, 86.8)
- added R10: 1k, Resistor_THT:R_Axial_DIN0204_L3.6mm_D1.6mm_P7.62mm_Horizontal, F.Cu at (113.2, 104.2)
- added R10: 1k, Resistor_THT:R_Axial_DIN0204_L3.6mm_D1.6mm_P7.62mm_Horizontal, F.Cu at (114.0, 218.5)
- added R11: 1k, Resistor_THT:R_Axial_DIN0204_L3.6mm_D1.6mm_P7.62mm_Horizontal, F.Cu at (113.2, 110.6)
- added R11: 1k, Resistor_THT:R_Axial_DIN0204_L3.6mm_D1.6mm_P7.62mm_Horizontal, F.Cu at (114.0, 224.9)
- added R12: 1k, Resistor_THT:R_Axial_DIN0204_L3.6mm_D1.6mm_P7.62mm_Horizontal, F.Cu at (113.2, 117.7)
- added R12: 1k, Resistor_THT:R_Axial_DIN0204_L3.6mm_D1.6mm_P7.62mm_Horizontal, F.Cu at (114.0, 232.0)
- added R2: 4k7, Resistor_THT:R_Axial_DIN0204_L3.6mm_D1.6mm_P7.62mm_Horizontal, F.Cu at (110.4, 75.6)
- added R3: 4k7, Resistor_THT:R_Axial_DIN0204_L3.6mm_D1.6mm_P7.62mm_Horizontal, F.Cu at (110.4, 65.1)
- added R4: 4k7, Resistor_THT:R_Axial_DIN0204_L3.6mm_D1.6mm_P7.62mm_Horizontal, F.Cu at (110.5, 54.1)
- added R5: 4k7, Resistor_THT:R_Axial_DIN0204_L3.6mm_D1.6mm_P7.62mm_Horizontal, F.Cu at (99.5, 51.0)
- added R6: 4k7, Resistor_THT:R_Axial_DIN0204_L3.6mm_D1.6mm_P7.62mm_Horizontal, F.Cu at (89.2, 51.0)
- added R7: 4k7, Resistor_THT:R_Axial_DIN0204_L3.6mm_D1.6mm_P7.62mm_Horizontal, F.Cu at (78.7, 51.1)
- added R8: 4k7, Resistor_THT:R_Axial_DIN0204_L3.6mm_D1.6mm_P7.62mm_Horizontal, F.Cu at (67.8, 51.2)
- added R9: 1k, Resistor_THT:R_Axial_DIN0204_L3.6mm_D1.6mm_P7.62mm_Horizontal, F.Cu at (114.0, 213.1)
- added R9: 1k, Resistor_THT:R_Axial_DIN0204_L3.6mm_D1.6mm_P7.62mm_Horizontal, F.Cu at (113.2, 98.8)
- added REF**: KiCad-Logo2_5mm_SilkScreen, Symbol:KiCad-Logo2_5mm_SilkScreen, F.Cu at (52.3, 122.8)
- added REF**: OSHW-Logo2_9.8x8mm_SilkScreen, Symbol:OSHW-Logo2_9.8x8mm_SilkScreen, F.Cu at (74.1, 188.5)
- added REF**: KiCad-Logo2_5mm_SilkScreen, Symbol:KiCad-Logo2_5mm_SilkScreen, F.Cu at (53.1, 237.1)
- added REF**: OSHW-Logo2_9.8x8mm_SilkScreen, Symbol:OSHW-Logo2_9.8x8mm_SilkScreen, F.Cu at (73.3, 74.2)
- added SW1: SW_Push, Button_Switch_THT:SW_PUSH_6mm, F.Cu at (123.1, 77.2)
- added SW2: SW_Push, Button_Switch_THT:SW_PUSH_6mm, F.Cu at (123.1, 66.9)
- added SW3: SW_Push, Button_Switch_THT:SW_PUSH_6mm, F.Cu at (123.1, 55.9)
- added SW4: SW_Push, Button_Switch_THT:SW_PUSH_6mm, F.Cu at (123.1, 45.3)
- A1: footprint Module:RaspberryPi_Pico_SMD_HandSolder -> Module:RaspberryPi_Pico_Common_THT
- Alimentación1: renamed from J11; footprint Connector_BarrelJack:BarrelJack_Horizontal -> Connector_BarrelJack:BarrelJack_CUI_PJ-079BH_Horizontal
- IA1: renamed from J12; value ID2 -> IA2
- moved R1 158.2 mm to (111.2, 201.1)
- moved ID1 157.3 mm to (138.3, 191.4), turned to 90 degrees
- moved R8 150.4 mm to (68.6, 165.5), turned to 0 degrees
- moved SW1 150.1 mm to (123.8, 191.6)
- moved R2 147.8 mm to (111.2, 189.9)
- moved R7 143.9 mm to (79.5, 165.4), turned to 0 degrees
- moved OD1 139.9 mm to (65.0, 236.9)
- moved R3 138.1 mm to (111.2, 179.4)
- moved R6 137.9 mm to (90.0, 165.3), turned to 0 degrees
- moved SW2 136.7 mm to (123.8, 181.2)
- moved A1 136.2 mm to (47.1, 230.6)
- moved ID2 132.4 mm to (138.5, 173.9), turned to 90 degrees
- moved R5 132.2 mm to (100.3, 165.3), turned to 0 degrees
- moved R4 128.2 mm to (111.3, 168.4)
- moved Alimentación1 125.9 mm to (132.6, 199.7), turned to 90 degrees
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- renumbered J2 to ID1, J3 to ID2, J4 to ID3, J5 to ID4, J6 to ID5, J7 to ID6, J8 to ID7, J9 to ID8, J1 to OD1
Connections:
- A1 pad 32: unconnected-(A1-GPIO27_ADC1-Pad32) -> GPIO27
- A1 pad 34: unconnected-(A1-GPIO28_ADC2-Pad34) -> GPIO28
- IA1 pad 2: GPIO26 -> GPIO28
- ID3 pad 2: /GPIO14 -> /GPIO16
- ID4 pad 2: /GPIO15 -> /GPIO17
- ID5 pad 2: /GPIO16 -> /GPIO18
- ID6 pad 2: /GPIO17 -> /GPIO19
- ID7 pad 2: /GPIO18 -> GPIO20
- ID8 pad 2: /GPIO19 -> GPIO21
- R3 pad 1: /GPIO14 -> /GPIO16
- R4 pad 1: /GPIO15 -> /GPIO17
- R5 pad 1: /GPIO16 -> /GPIO18
- R6 pad 1: /GPIO17 -> /GPIO19
- R7 pad 1: /GPIO18 -> GPIO20
- R8 pad 1: /GPIO19 -> GPIO21
- SW3 pad 1: /GPIO14 -> /GPIO16
- SW4 pad 1: /GPIO15 -> /GPIO17
Routing:
- net /Vsys: track 0.00 -> 1135.6 mm
- net /GPIO17: track 0.00 -> 202.0 mm
- net /GPIO13: track 0.00 -> 199.1 mm
- net /GPIO16: track 0.00 -> 183.5 mm
- net /GPIO12: track 0.00 -> 163.3 mm
- net GPIO21: track 0.00 -> 155.5 mm
- net /GPIO18: track 0.00 -> 147.4 mm
- net GPIO20: track 0.00 -> 139.9 mm
- net /GPIO19: track 0.00 -> 137.4 mm
- net GPIO28: track 0.00 -> 106.6 mm
- net Net-(J14-Pin_1): track 0.00 -> 99.2 mm
- net Net-(J13-Pin_1): track 0.00 -> 96.5 mm
- net GPIO26: track 0.00 -> 53.6 mm
- net GPIO27: track 0.00 -> 44.3 mm
- net /GPIO14: track 0.00 -> 44.3 mm
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- added copper zone on B.Cu, net GND
Other:
- board outline added: 100.8 x 214.3 mm
- board text added: "Entrada analógica"
- board text added: "Entradas Digitales"
- board text added: "Open PLC - Pico 2"
- board text added: "Salida I2C"
- board text added: "Salidas Digitales"
- board text added: "Salidas analógicas"
- board text added: "~"
